Commit message: Create launch file

File: install/arduinobot_description/share/arduinobot_description/urdf/arduinobot.urdf.xacro (robot description, xacro)
@@ -88,5 +88,5 @@
             <origin rpy="0 0 -${PI/2}" xyz="-0.04 0.5 -0.1"/>
             <geometry>
-                <mesh filename= "package://arduinobot_description/meshes/right_finger.STL" scale = "0.01 0.01 0.01"/>
+                <mesh filename= "package://arduinobot_description/meshes/left_finger.STL" scale = "0.01 0.01 0.01"/>
             </geometry>
         </visual>

Commit message: Add RGB camera

File: install/arduinobot_description/share/arduinobot_description/urdf/arduinobot.urdf.xacro (robot description, xacro)
@@ -107,3 +107,16 @@
         <mimic joint="joint_4" multiplier="-1"/>
     </joint>
+    <link name="rgb_camera">
+        <visual>
+            <origin rpy="-1.57 0 -1.57" xyz="-0.1 0.125 0"/>
+            <geometry>
+                <mesh filename = "package://arduinobot_description/meshes/pi_camera.STL" scale = "0.01 0.01 0.01"/>
+            </geometry>
+        </visual>
+    </link>
+    <joint name = "rgb_camera_joint" type="fixed">
+        <parent link ="base_link"/>
+        <child link = "rgb_camera"/>
+        <origin rpy = "-0.5 0 1.57" xyz ="0 0.45 0.2"/>
+    </joint>
 </robot>

Commit message: rgb-connected

File: install/arduinobot_description/share/arduinobot_description/urdf/arduinobot.urdf.xacro (robot description, xacro)
@@ -4,6 +4,15 @@
     <xacro:property name="effort" value="30.0"/>
     <xacro:property name="velocity" value="10.0"/>
+    <xacro:macro name = "default_inertial" params="mass">
+        <inertial>
+            <mass value="${mass}"/>
+            <inertia ixx="1.0" ixy="0.0" ixz="0.0"
+                     iyy="1.0" iyz="0.0"
+                     izz="1.0"/>
+        </inertial>
+    </xacro:macro>
     <link name = "world"/>
     <link name = "base_link">
+        <xacro:default_inertial mass="1.0"/>
         <visual>
             <origin rpy = "0 0 0" xyz = "-0.5 -0.5 0"/>
@@ -12,4 +21,10 @@
             </geometry>
         </visual>
+        <collision>
+            <origin rpy = "0 0 0" xyz = "-0.5 -0.5 0"/>
+            <geometry>
+                <mesh filename = "package://arduinobot_description/meshes/basement.STL" scale = "0.01 0.01 0.01" />
+            </geometry>
+        </collision>
     </link>
     <joint name = "virtual_joint" type = "fixed">
@@ -19,4 +34,5 @@
     </joint>
     <link name = "base_plate">
+        <xacro:default_inertial mass="0.1"/>
         <visual>
             <origin rpy = "0 0 0" xyz = "-0.39 -0.39 -0.56"/>
@@ -25,4 +41,10 @@
             </geometry>
         </visual>
+        <collision>
+            <origin rpy = "0 0 0" xyz = "-0.39 -0.39 -0.56"/>
+            <geometry>
+                <mesh filename = "package://arduinobot_description/meshes/base_plate.STL" scale = "0.01 0.01 0.01"/>
+            </geometry>
+        </collision>
     </link>
     <joint name = "joint_1" type = "revolute">
@@ -34,4 +56,5 @@
     </joint>
     <link name="forward_drive_arm">
+        <xacro:default_inertial mass="0.1"/>
         <visual>
             <origin rpy = "0 -${PI/2} ${PI/2}" xyz = "0.19 0.06 -0.08"/>
@@ -40,4 +63,10 @@
             </geometry>
         </visual>
+        <collision>
+            <origin rpy = "0 -${PI/2} ${PI/2}" xyz = "0.19 0.06 -0.08"/>
+            <geometry>
+                <mesh filename = "package://arduinobot_description/meshes/forward_drive_arm.STL" scale = "0.01 0.01 0.01"/>
+            </geometry>
+        </collision>
     </link>
     <joint name = "joint2" type="revolute">
@@ -49,4 +78,5 @@
     </joint>
     <link name="horizontal_arm">
+        <xacro:default_inertial mass="0.1"/>
         <visual>
             <origin rpy = "${PI/2} 0 ${PI/2}" xyz = "-0.03 -0.4 -0.06"/>
@@ -55,4 +85,10 @@
             </geometry>
         </visual>
+        <collision>
+            <origin rpy = "${PI/2} 0 ${PI/2}" xyz = "-0.03 -0.4 -0.06"/>
+            <geometry>
+                <mesh filename = "package://arduinobot_description/meshes/horizontal_arm.STL" scale = "0.01 0.01 0.01"/>
+            </geometry>
+        </collision>
     </link>
     <joint name = "joint3" type="revolute">
@@ -64,4 +100,5 @@
     </joint>
     <link name="claw_support">
+        <xacro:default_inertial mass="0.05"/>
         <visual>
             <origin rpy = "0 0 ${PI/2}" xyz ="0 -0.05 -0.15"/>
@@ -70,4 +107,10 @@
             </geometry>
         </visual>
+        <collision>
+            <origin rpy = "0 0 ${PI/2}" xyz ="0 -0.05 -0.15"/>
+            <geometry>
+                <mesh filename = "package://arduinobot_description/meshes/claw_support.STL" scale = "0.01 0.01 0.01"/>
+            </geometry>
+        </collision>
     </link>
     <joint name = "horizontal_arm_to_claw_support" type="fixed">
@@ -77,4 +120,5 @@
     </joint>
     <link name="gripper_right">
+        <xacro:default_inertial mass="0.05"/>
         <visual>
             <origin rpy="0 0 -${PI/2}" xyz="-0.1 0.5 -0.1"/>
@@ -83,6 +127,13 @@
             </geometry>
         </visual>
+        <collision>
+            <origin rpy="0 0 -${PI/2}" xyz="-0.1 0.5 -0.1"/>
+            <geometry>
+                <mesh filename= "package://arduinobot_description/meshes/right_finger.STL" scale = "0.01 0.01 0.01"/>
+            </geometry>
+        </collision>
     </link>
     <link name="gripper_left">
+        <xacro:default_inertial mass="0.05"/>
         <visual>
             <origin rpy="0 0 -${PI/2}" xyz="-0.04 0.5 -0.1"/>
@@ -91,4 +142,10 @@
             </geometry>
         </visual>
+        <collision>
+            <origin rpy="0 0 -${PI/2}" xyz="-0.04 0.5 -0.1"/>
+            <geometry>
+                <mesh filename= "package://arduinobot_description/meshes/left_finger.STL" scale = "0.01 0.01 0.01"/>
+            </geometry>
+        </collision>
     </link>
     <joint name="joint_4" type="revolute">
@@ -109,14 +166,60 @@
     <link name="rgb_camera">
         <visual>
-            <origin rpy="-1.57 0 -1.57" xyz="-0.1 0.125 0"/>
+            <origin rpy="-1.57 0 -1.57" xyz="-0.1 0.125 0.15"/>
             <geometry>
                 <mesh filename = "package://arduinobot_description/meshes/pi_camera.STL" scale = "0.01 0.01 0.01"/>
             </geometry>
         </visual>
-    </link>
+        <collision>
+            <geometry>
+              <box size="0.05 0.05 0.05"/> <!-- Approximate volume -->
+            </geometry>
+            <origin rpy="-1.57 0 -1.57" xyz="-0.1 0.125 0.15"/>
+          </collision>
+          <inertial>
+            <mass value="0.001"/>
+            <origin xyz="0 0 0" rpy="0 0 0"/>
+            <inertia ixx="1e-6" ixy="0" ixz="0" iyy="1e-6" iyz="0" izz="1e-6"/>
+          </inertial>
+    </link>
+    <gazebo reference="rgb_camera">
+        <sensor name="camera" type="camera">
+            <always_on>true</always_on>
+            <update_rate>30.0</update_rate>
+            <visualize>true</visualize>
+            <topic>/image_raw</topic>
+            <gz_frame_id>/rgb_camera</gz_frame_id>
+            <camera name="camera">
+              <horizontal_fov>1.21126</horizontal_fov>
+              <image>
+                <width>2304</width>
+                <height>1296</height>
+                <format>R8G8B8</format>
+              </image>
+              <distortion>
+                <k1>0.0</k1>
+                <k2>0.0</k2>
+                <k3>0.0</k3>
+                <p1>0.0</p1>
+                <p2>0.0</p2>
+                <center>0.5 0.5</center>
+              </distortion>
+            </camera>
+        </sensor>
+    </gazebo>
+    <gazebo>
+        <!-- ROS 2 Humble -->
+        <xacro:if value="$(arg is_ignition)">
+          <plugin filename="ign_ros2_control-system" name="ign_ros2_control::IgnitionROS2ControlPlugin">
+          </plugin>
+          <plugin filename="ignition-gazebo-sensors-system" name="ignition::gazebo::systems::Sensors">
+            <render_engine>ogre2</render_engine>
+          </plugin>
+        </xacro:if>
+      </gazebo>
     <joint name = "rgb_camera_joint" type="fixed">
         <parent link ="base_link"/>
         <child link = "rgb_camera"/>
-        <origin rpy = "-0.5 0 1.57" xyz ="0 0.45 0.2"/>
+        <origin xyz="0 0.45 0.2" rpy="0 -0.5 1.57"/>
     </joint>
 </robot>

Commit message: controller-interface

File: install/arduinobot_description/share/arduinobot_description/urdf/arduinobot.urdf.xacro (robot description, xacro)
@@ -1,4 +1,8 @@
 <?xml version = "1.0"?>
 <robot xmlns:xacro = "http://www.ros.org/wiki/xacro" name = "arduinobot">
+    <xacro:arg name = "is_ignition" default = "true"/>
+    <xacro:include filename="$(find arduinobot_description)/urdf/arduinobot_gazebo.xacro"/>
+    <xacro:include filename="$(find arduinobot_description)/urdf/arduinobot_ros2_control.xacro"/>
+    <!-- Useful Macros-->
     <xacro:property name="PI" value="3.14159"/>
     <xacro:property name="effort" value="30.0"/>
@@ -70,5 +74,5 @@
         </collision>
     </link>
-    <joint name = "joint2" type="revolute">
+    <joint name = "joint_2" type="revolute">
         <parent link ="base_plate"/>
         <child link = "forward_drive_arm"/>
@@ -92,5 +96,5 @@
         </collision>
     </link>
-    <joint name = "joint3" type="revolute">
+    <joint name = "joint_3" type="revolute">
         <parent link ="forward_drive_arm"/>
         <child link = "horizontal_arm"/>
@@ -208,14 +212,4 @@
         </sensor>
     </gazebo>
-    <gazebo>
-        <!-- ROS 2 Humble -->
-        <xacro:if value="$(arg is_ignition)">
-          <plugin filename="ign_ros2_control-system" name="ign_ros2_control::IgnitionROS2ControlPlugin">
-          </plugin>
-          <plugin filename="ignition-gazebo-sensors-system" name="ignition::gazebo::systems::Sensors">
-            <render_engine>ogre2</render_engine>
-          </plugin>
-        </xacro:if>
-      </gazebo>
     <joint name = "rgb_camera_joint" type="fixed">
         <parent link ="base_link"/>
